File: PCB/harp expander.sch (EAGLE design)
At the start: 126 parts, among them IC1 XMEGA-A1TQFP, IC10 74AHC1G125DBV, IC11 74AHC1G125DBV, IC12 74AHC1G125DBV, IC13 74AHC1G125DBV, IC14 74AHC1G125DBV, IC15 74AHC1G125DBV, IC16 74AHC1G125DBV, IC2 USBLC6-2SC6, IC3 FT232RL, IC4 TLV70033DDCR, IC5 TLV70033DDCR, IC6 SI8610BC-B-IS, IC7 74AHC1G125DBV, IC8 74AHC1G125DBV, IC9 74AHC1G125DBV, T10 BC850, T11 BC850, T12 BC850, T13 BC850, T2 BC850, T3 BC850, T4 BC850, T5 BC850, T6 BC850, T7 BC850, T8 BC850, T9 BC850

Commit message: Updated design files to the latest version.
Parts:
- removed C35, C36: 100nF, rcl:C-EUC0402
- removed IC10, IC11, IC12, IC13, IC15, IC16, IC8, IC9: 74AHC1G125DBV, 74xx-little-de:74AHC1G125DBV
- added GND_TP0, GND_TP1: TPPAD1-13, testpad:TPPAD1-13
- added R18, R19, R38, R43, R46, R47: 10k, rcl:R-EU_R0402
- added R48, R49, R50, R51, R52: 100R, rcl:R-EU_R0603
- added R53: 1k, rcl:R-EU_R0402
- added U1, U2: 744245X, harp input expander:744245X
- BNC0, BNC1, BNC2, BNC3, BNC4: value (none) -> BNC plug; MPN (none) -> 73100-0105
- C1, C12, C13, C14, C15, C16, C17, C18, C19, C20, C21, C22, C25, C26, C27, C28, C29, C3, C30, C31, C32, C5, C7, C9: MPN (none) -> MC0402B104K160CT
- C10, C11, C23, C24: MPN (none) -> C1608X6S1C475K080AC
- C2: MPN (none) -> 885012205084
- C33, C34, C37, C38: value 100nF -> 4.7uF; device rcl:C-EUC0402 -> rcl:C-EUC0603; MPN (none) -> C1608X6S1C475K080AC
- C4, C6: MPN (none) -> 04025A470JAT2A
- C8: MPN (none) -> TAJA475K016UNJ
- CLKIN, CLKOUT: value STEREO_JACK -> CLCK_JACK; MPN (none) -> 35RASMT2BHNTRX
- IC1: MPN (none) -> ATXMEGA128A1U-AU
- IC14, IC7: value 74AHC1G125DBV -> SN74LVC1G125DBVT; MPN (none) -> SN74LVC1G125DBVT
- IC2: MPN (none) -> USBLC6-2SC6
- IC3: device ftdichip:FT232RL -> harp input expander:FT232RL; MPN (none) -> FT232RL-REEL
- IC4, IC5: MPN (none) -> TLV70033DDCR
- IC6: MPN (none) -> SI8610EC-B-IS
- JP1: value (none) -> CLCK Jumper; MPN (none) -> 42375-1856
- L1: value ??? -> 40R@100MHz; MPN (none) -> MI0805K400R-10
- LED0, LED1, LED2, LED3, LED4, LED5: MPN (none) -> 5690-111-100F
- OSC: value OSCILLATOR -> Oscillator; MPN (none) -> DSC1001CI5-032.0000T
- PDI: value (none) -> PROG HEADER; device con-lstb:MA03-2 -> harp input expander:MA03-2; MPN (none) -> 67996-206HLF
- R1: MPN (none) -> CRCW04021M00FKED
- R10, R11, R12, R13, R14, R15, R3, R9: value 100k -> 10k; MPN (none) -> CRCW040210K0FKED
- R16, R17: MPN (none) -> CRCW040210K0FKED
- R2: value 10 -> 10R; MPN (none) -> CRCW040210R0FKEDHP
- R20, R21, R22, R23, R24, R25, R26, R27, R28, R29, R30, R31: MPN (none) -> CRCW04021K00FKED
- R32, R33, R34, R35, R36, R37, R39, R40, R41, R42, R44, R45: value 330 -> 330R; MPN (none) -> RC0402FR-07330RL
- R4, R5, R6, R7, R8: value 100k -> 100R; device rcl:R-EU_R0402 -> rcl:R-EU_R0603; MPN (none) -> CRCW0603100RFKEAHP
- SV1: value (none) -> I/O Header; device con-ml:ML10L -> harp input expander:ML10L; MPN (none) -> SBH11-PBPC-D05-RA-BK
- T10, T11, T12, T13, T2, T3, T4, T5, T6, T7, T8, T9: MPN (none) -> BC850C,215
- USB: value USB_MINI_B -> mini USB; MPN (none) -> UX60-MB-5S8
Connections:
- removed net EXT_I5: IC12A.I, R9.1, SV1.1
- removed net EXT_I6: IC13A.I, R10.1, SV1.2
- removed net EXT_I7: IC14A.I, R11.1, SV1.3
- removed net EXT_I8: IC15A.I, R12.1, SV1.4
- removed net EXT_I9: IC16A.I, R13.1, SV1.5
- removed net I0: IC1.PD0(OC0A/SDA), IC7A.O
- removed net I1: IC1.PD1(OC0B/XCK0/SCL), IC8A.O
- removed net I2: IC1.PD2(OC0C/RXD0), IC9A.O
- removed net I3: IC1.PD3(OC0D/TXD0), IC10A.O
- removed net I4: IC1.PD4(OC1A/!SS!), IC11A.O
- removed net I5: IC1.PD5(OC1B/XCK1/MOSI), IC12A.O
- removed net I6: IC1.PD6(RXD1/MISO), IC13A.O
- removed net I7: IC1.PD7(TXD1/SCK/CLKO/EVO), IC14A.O
- removed net I8: IC1.PE0(OC0A/SDA), IC15A.O
- removed net I9: IC1.PE1(OC0B/XCK0/SCL), IC16A.O
- removed net N$10: BNC3.1, IC10A.I, R7.1
- removed net N$11: BNC4.1, IC11A.I, R8.1
- removed net N$12: BNC0.1, IC7A.I, R4.1
- removed net N$45: R16.1, SV1.6
- removed net N$46: R17.1, SV1.7
- new net BNC_IOS_DIR: IC1.PD7(TXD1/SCK/CLKO/EVO), U2.DIR
- new net BNC_IOS_ENBL: IC1.PD6(RXD1/MISO), R15.2, U2.OE
- new net IDE_IOS_DIR: IC1.PB5(ADCB5/TDI), U1.DIR
- new net IDE_IOS_ENBL: IC1.PB6(ADCB6/TCK), R14.2, U1.OE
- new net IO0: BNC0.1, R19.2, R4.1
- new net IO1: BNC1.1, R38.2, R5.1
- new net IO2: BNC2.1, R43.2, R6.1
- new net IO3: BNC3.1, R46.2, R7.1
- new net IO4: BNC4.1, R47.2, R8.1
- new net IO5: R48.1, R9.1, SV1.1
- new net IO6: R10.1, R49.1, SV1.2
- new net IO7: R11.1, R50.1, SV1.3
- new net IO8: R12.1, R51.1, SV1.4
- new net IO9: R13.1, R52.1, SV1.5
- new net IO_BUTTON0: IC14A.I, R16.1, SV1.6
- new net IO_BUTTON1: IC7A.I, R17.1, SV1.7
- new net N$114: R52.2, U1.A4
- new net N$115: R4.2, U2.A0
- new net N$116: R5.2, U2.A1
- new net N$122: R6.2, U2.A2
- new net N$142: R7.2, U2.A3
- new net N$152: R8.2, U2.A4
- new net N$175: IC3.!RESET, R18.2
- new net N$68: R49.2, U1.A1
- new net N$69: R50.2, U1.A2
- new net N$97: R51.2, U1.A3
- new net PD0: IC1.PD0(OC0A/SDA), U2.B4
- new net PD1: IC1.PD1(OC0B/XCK0/SCL), U2.B3
- new net PD2: IC1.PD2(OC0C/RXD0), U2.B2
- new net PD3: IC1.PD3(OC0D/TXD0), U2.B1
- new net PD4: IC1.PD4(OC1A/!SS!), U2.B0
- new net PE0: IC1.PC0(OC0A/SDA), U1.B0
- new net PE1: IC1.PC1(OC0B/XCK0/SCL), U1.B1
- new net PE2: IC1.PC2(OC0C/RXD0), U1.B2
- new net PE3: IC1.PC3(OC0D/TXD0), U1.B3
- new net PE4: IC1.PC4(OC1A/!SS!), U1.B4
- net +3V3: now also R18.1, U1.VCC_B, U2.VCC_B; no longer C27.1, C28.1, C35.1, C36.1, IC10P.VCC, IC11P.VCC, IC12P.VCC, IC13P.VCC, IC15P.VCC, IC16P.VCC, IC8P.VCC, IC9P.VCC, R14.2, R15.2, SV1.8
- net +5V: now also C27.1, C28.1, C37.1, C38.1, U1.VCC_A, U2.VCC_A
- net GND: now also GND_TP0.TP, GND_TP1.TP, R14.1, R15.1, R16.2, R17.2, R19.1, R38.1, R43.1, R46.1, R47.1, R53.2, U1.GND, U2.GND; no longer C35.2, C36.2, IC10A.OE, IC10P.GND, IC11A.OE, IC11P.GND, IC12A.OE, IC12P.GND, IC13A.OE, IC13P.GND, IC15A.OE, IC15P.GND, IC16A.OE, IC16P.GND, IC8A.OE, IC8P.GND, IC9A.OE, IC9P.GND, R4.2, R5.2, R6.2, R7.2, R8.2
- net N$6: now also R48.2, U1.A0; no longer BNC1.1, IC8A.I, R5.1
- net N$9: now also IC1.PE3(OC0D/TXD0), R53.1; no longer BNC2.1, IC9A.I, R6.1
- net USER_BUTTON_0: now also IC1.PA1(ADCA1), IC14A.O; no longer C37.1, IC1.PA0(ADCA0/AREFA), R14.1, R16.2
- net USER_BUTTON_1: now also IC1.PA0(ADCA0/AREFA), IC7A.O; no longer C38.1, IC1.PA1(ADCA1), R15.1, R17.2
Other:
- note added: "u IO-function selection"
- note removed: "TLV70033DDC 200mA 0.24€ LD1117S33TR 800mA 0.30€ TLV74333PDBVR 300mA 0.20€"
- moved on the sheet: BNC0, BNC1, BNC2, BNC3, BNC4, C27, C28, C29, C30, C31, C32, C33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
