File: PCB modules/servo driver/harp expander servo driver v1.0.brd (EAGLE design)
At the start: 70 x 46 mm, 28 parts, among them U1 SI8641AB-B-IS1R, U2 SI8641AB-B-IS1R, U3 LT1765, U4 NCP718XSN500, X1 CON_3.5MM_1X3, X2 CON_3.5MM_1X3, X3 CON_3.5MM_1X3, X4 aux_header, X5 2510-

Commit message: Minor updates.
Parts:
- D1: value MBRM120 -> BAT42W
