File: PCB modules/servo driver/harp expander servo driver v1.0.sch (EAGLE design)
At the start: 28 parts, among them U1 SI8641AB-B-IS1R, U2 SI8641AB-B-IS1R, U3 LT1765, U4 NCP718XSN500, X1 CON_3.5MM_1X3, X2 CON_3.5MM_1X3, X3 CON_3.5MM_1X3, X4 aux_header, X5 2510-

Commit message: Minor updates.
Parts:
- C1, C2, C3, C4, C5, C6: DIGIKEY_PN (none) -> 445-6899-2-ND; MPN MC0402B104K160CT -> CGA2B3X7R1H104K050BB
- C10: DIGIKEY_PN (none) -> 587-3238-1-ND; MPN GRM188R61A106ME69D -> EMK107BBJ106MA-T
- C11: DIGIKEY_PN (none) -> 1276-1184-1-ND; MPN ?? 1u -> CL10B105KA8NNNC
- C7: DIGIKEY_PN (none) -> 490-12738-1-ND; MPN GRM188R61E225MA12D -> GRM188R61E225MA12D
- C8: DIGIKEY_PN (none) -> 1276-1532-6-ND; MPN VJ0402Y222KXJCW1BC -> CL05B222JB5NNNC
- C9: DIGIKEY_PN (none) -> 490-GCG188R91H184KA01DCT-ND; MPN GRM188R71E184KA88D -> GCG188R91H184KA01D
- D1: value MBRM120 -> BAT42W; DIGIKEY_PN (none) -> BAT42W-E3-08CT-ND; MPN MBRM120LT3G -> BAT42W-E3-08
- D2: DIGIKEY_PN (none) -> 1514-CMDSH-3TRPBFREECT-ND; MPN CMDSH-3 TR PBFREE -> CMDSH-3
- D3: DIGIKEY_PN (none) -> SSB43L-E3/52TGICT-ND; MPN (none) -> SSB43L-E3/52T; VALUE2 (none) -> DIODE SCHOTTKY 30V 4A DO214AA
- L1: DESCRPT Fixed Inductors 2.6uH 30% SMD 5028 -> (none); DIGIKEY_PN (none) -> SRR5028-2R6YCT-ND; MOUSER 652-SRR5028-2R6Y -> (none); MOUSER_PN (none) -> 652-SRR5028-2R6Y; MPN (none) -> SRR5028-2R6Y; VALUE2 2.6uL 1A -> 2.6uH 3A
- PWR1: DIGIKEY_PN (none) -> 163-179PH-EX MOUSER; MPN (none) -> 163-179PH-EX
- R1: DIGIKEY_PN (none) -> 311-40.2KLRCT-ND; MPN CRCW040240K2FKED -> RC0402FR-0740K2L
- R2, R3: DIGIKEY_PN (none) -> 541-3959-1-ND; MPN CRCW040210K0FKED -> CRCW040210K0FKEDC
- U1, U2: DIGIKEY_PN (none) -> 336-5212-1-ND; MOUSER_PN (none) -> 634-SI8641AB-B-IS1R; MPN (none) -> SI8641AB-B-IS1R
- U3: DESCRIPTION (none) -> Buck Switching Regulator Output 3A; DIGIKEY_PN (none) -> LT1765EFE#TRPBFCT-ND; MPN (none) -> LT1765EFE#TRPBF
- U4: DIGIKEY_PN (none) -> NCP718BSN500T1GOSCT-ND; MPN (none) -> NCP718BSN500T1G
- X1, X2, X3: DIGIKEY_PN (none) -> 732-2770-ND; MPN (none) -> 691322110003
- X4: MPN (none) -> n.a.
- X5: DIGIKEY_PN (none) -> S9169-ND
