File: PCB modules/servo driver/harp expander servo driver v1.1.brd (EAGLE design)
At the start: 70 x 46 mm, 28 parts, among them U1 SI8641AB-B-IS1R, U2 SI8641AB-B-IS1R, U3 LT1765, U4 NCP718XSN500, X1 CON_3.5MM_1X3, X2 CON_3.5MM_1X3, X3 CON_3.5MM_1X3, X4 aux_header, X5 2510-

Commit message: Added filtering on inputs and reset lines to prevent erroneous behavior in noisy environments.
Parts:
- added EXTERNAL_1, EXTERNAL_2, EXTERNAL_3: TERMINAL BLOCK PLUG 3WAY, harp expander servo driver v1.0:-
- added EXTERNAL_4, EXTERNAL_5: CNTR PLRZD RECPT 10P, harp expander servo driver v1.0:-
- added EXTERNAL_6: 10 COND. 28AWG ROUND 1PC=100FT, harp expander servo driver v1.0:-
- X5: value 2510- -> IDC 10WAY STRAIGHT
Changed lines of the file:
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@@
 <?xml version="1.0" encoding="utf-8"?>
 <!DOCTYPE eagle SYSTEM "eagle.dtd">
-<eagle version="9.5.1">
+<eagle version="9.6.2">
 <drawing>
 <settings>
@@
 <layer number="14" name="Route14" color="1" fill="6" visible="no" active="no"/>
 <layer number="15" name="Route15" color="4" fill="6" visible="no" active="no"/>
-<layer number="16" name="Bottom" color="1" fill="1" visible="no" active="yes"/>
+<layer number="16" name="Bottom" color="1" fill="1" visible="yes" active="yes"/>
 <layer number="17" name="Pads" color="2" fill="1" visible="yes" active="yes"/>
 <layer number="18" name="Vias" color="2" fill="1" visible="yes" active="yes"/>
@@
 <attribute name="VALUE" x="44.4174" y="29.1632" size="1.27" layer="27" rot="R270"/>
 </element>
-<element name="X5" library="con-3m" library_urn="urn:adsk.eagle:library:119" package="PAK100/2500-10" package3d_urn="urn:adsk.eagle:package:5571/1" value="2510-" x="23.419" y="39.2992" locked="yes" smashed="yes">
+<element name="X5" library="con-3m" library_urn="urn:adsk.eagle:library:119" package="PAK100/2500-10" package3d_urn="urn:adsk.eagle:package:5571/1" value="IDC 10WAY STRAIGHT" x="23.419" y="39.2992" locked="yes" smashed="yes">
 <attribute name="DIGIKEY_PN" value="S9169-ND" x="23.419" y="39.2992" size="1.778" layer="27" display="off"/>
 <attribute name="MF" value="-" x="23.419" y="39.2992" locked="yes" size="1.778" layer="27" display="off"/>
@@
 </element>
 <element name="U1" library="harp expander servo driver v1.0" package="SO16W" package3d_urn="urn:adsk.eagle:package:16487/2" value="SI8641AB-B-IS1R" x="12.4512" y="22.799" smashed="yes" rot="R180">
-<attribute name="DIGIKEY_PN" value="336-5212-1-ND" x="12.4512" y="22.799" size="1.778" layer="27" rot="R180" display="off"/>
+<attribute name="DIGIKEY_PN" value="SI8641AB-B-IS-ND" x="12.4512" y="22.799" size="1.778" layer="27" rot="R180" display="off"/>
 <attribute name="MOUSER_PN" value="634-SI8641AB-B-IS1R" x="12.4512" y="22.799" size="1.778" layer="27" rot="R180" display="off"/>
 <attribute name="MPN" value="SI8641AB-B-IS1R" x="12.4512" y="22.799" size="1.778" layer="27" rot="R180" display="off"/>
@@
 </element>
 <element name="U2" library="harp expander servo driver v1.0" package="SO16W" package3d_urn="urn:adsk.eagle:package:16487/2" value="SI8641AB-B-IS1R" x="26.9288" y="22.599" smashed="yes" rot="R180">
-<attribute name="DIGIKEY_PN" value="336-5212-1-ND" x="26.9288" y="22.599" size="1.778" layer="27" rot="R180" display="off"/>
+<attribute name="DIGIKEY_PN" value="SI8641AB-B-IS-ND" x="26.9288" y="22.599" size="1.778" layer="27" rot="R180" display="off"/>
 <attribute name="MOUSER_PN" value="634-SI8641AB-B-IS1R" x="26.9288" y="22.599" size="1.778" layer="27" rot="R180" display="off"/>
 <attribute name="MPN" value="SI8641AB-B-IS1R" x="26.9288" y="22.599" size="1.778" layer="27" rot="R180" display="off"/>
@@
 <attribute name="VALUE" x="54.491" y="18.049" size="1.27" layer="27" rot="R90"/>
 </element>
+<element name="EXTERNAL_1" library="harp expander servo driver v1.0" package="-" value="TERMINAL BLOCK PLUG 3WAY" x="3.2512" y="0.8128" smashed="yes">
+<attribute name="DIGIKEY_PN" value="732-2752-ND" x="3.2512" y="0.8128" size="1.778" layer="27" display="off"/>
+<attribute name="MPN" value="691361100003" x="3.2512" y="0.8128" size="1.778" layer="27" display="off"/>
+<attribute name="TYPE" value="-" x="3.2512" y="0.8128" size="1.778" layer="27" display="off"/>
+</element>
+<element name="EXTERNAL_2" library="harp expander servo driver v1.0" package="-" value="TERMINAL BLOCK PLUG 3WAY" x="3.2512" y="0.8128" smashed="yes">
+<attribute name="DIGIKEY_PN" value="732-2752-ND" x="2.4384" y="2.8448" size="1.778" layer="27" display="off"/>
+<attribute name="MPN" value="691361100003" x="3.2512" y="0.8128" size="1.778" layer="27" display="off"/>
+<attribute name="TYPE" value="-" x="3.2512" y="0.8128" size="1.778" layer="27" display="off"/>
+</element>
+<element name="EXTERNAL_3" library="harp expander servo driver v1.0" package="-" value="TERMINAL BLOCK PLUG 3WAY" x="3.2512" y="0.8128" smashed="yes">
+<attribute name="DIGIKEY_PN" value="732-2752-ND" x="2.4384" y="6.096" size="1.778" layer="27" display="off"/>
+<attribute name="MPN" value="691361100003" x="3.2512" y="0.8128" size="1.778" layer="27" display="off"/>
+<attribute name="TYPE" value="-" x="3.2512" y="0.8128" size="1.778" layer="27" display="off"/>
+</element>
+<element name="EXTERNAL_4" library="harp expander servo driver v1.0" package="-" value="CNTR PLRZD RECPT 10P" x="3.2512" y="0.8128" smashed="yes">
+<attribute name="DIGIKEY_PN" value="AKC10H-ND" x="2.4384" y="12.5984" size="1.778" layer="27" display="off"/>
+<attribute name="MPN" value="1658621-1" x="3.2512" y="0.8128" size="1.778" layer="27" display="off"/>
+<attribute name="TYPE" value="-" x="3.2512" y="0.8128" size="1.778" layer="27" display="off"/>
+</element>
+<element name="EXTERNAL_5" library="harp expander servo driver v1.0" package="-" value="CNTR PLRZD RECPT 10P" x="3.2512" y="0.8128" smashed="yes">
+<attribute name="DIGIKEY_PN" value="AKC10H-ND" x="2.4384" y="25.6032" size="1.778" layer="27" display="off"/>
+<attribute name="MPN" value="1658621-1" x="3.2512" y="0.8128" size="1.778" layer="27" display="off"/>
+<attribute name="TYPE" value="-" x="3.2512" y="0.8128" size="1.778" layer="27" display="off"/>
+</element>
+<element name="EXTERNAL_6" library="harp expander servo driver v1.0" package="-" value="10 COND. 28AWG ROUND 1PC=100FT" x="3.2512" y="0.8128" smashed="yes">
+<attribute name="DIGIKEY_PN" value="3M157849-100-ND" x="2.4384" y="51.6128" size="1.778" layer="27" display="off"/>
+<attribute name="MPN" value="3365/10 100" x="3.2512" y="0.8128" size="1.778" layer="27" display="off"/>
+<attribute name="TYPE" value="-" x="3.2512" y="0.8128" size="1.778" layer="27" display="off"/>
+</element>
 </elements>
