File: PCB modules/servo driver/harp expander servo driver v1.1.sch (EAGLE design)
At the start: 28 parts, among them U1 SI8641AB-B-IS1R, U2 SI8641AB-B-IS1R, U3 LT1765, U4 NCP718XSN500, X1 CON_3.5MM_1X3, X2 CON_3.5MM_1X3, X3 CON_3.5MM_1X3, X4 aux_header, X5 2510-

Commit message: Added filtering on inputs and reset lines to prevent erroneous behavior in noisy environments.
Parts:
- added EXTERNAL_1, EXTERNAL_2, EXTERNAL_3: TERMINAL BLOCK PLUG 3WAY, harp expander servo driver v1.0:EXTERNAL
- added EXTERNAL_4, EXTERNAL_5: CNTR PLRZD RECPT 10P, harp expander servo driver v1.0:EXTERNAL
- added EXTERNAL_6: 10 COND. 28AWG ROUND 1PC=100FT, harp expander servo driver v1.0:EXTERNAL
- U1, U2: DIGIKEY_PN 336-5212-1-ND -> SI8641AB-B-IS-ND
- X5: value 2510- -> IDC 10WAY STRAIGHT
Changed lines of the file:
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@@
 <?xml version="1.0" encoding="utf-8"?>
 <!DOCTYPE eagle SYSTEM "eagle.dtd">
-<eagle version="9.5.1">
+<eagle version="9.6.2">
 <drawing>
 <settings>
@@
 <attribute name="VALUE2" value="+6.35V"/>
 </part>
-<part name="X5" library="con-3m" library_urn="urn:adsk.eagle:library:119" deviceset="2510-" device="" package3d_urn="urn:adsk.eagle:package:5571/1">
+<part name="X5" library="con-3m" library_urn="urn:adsk.eagle:library:119" deviceset="2510-" device="" package3d_urn="urn:adsk.eagle:package:5571/1" value="IDC 10WAY STRAIGHT">
 <attribute name="DIGIKEY_PN" value="S9169-ND"/>
 <attribute name="MF" value="-"/>
@@
 </part>
 <part name="U1" library="harp expander servo driver v1.0" deviceset="SI8641AB" device="W" package3d_urn="urn:adsk.eagle:package:16487/2" value="SI8641AB-B-IS1R">
-<attribute name="DIGIKEY_PN" value="336-5212-1-ND"/>
+<attribute name="DIGIKEY_PN" value="SI8641AB-B-IS-ND"/>
 <attribute name="MOUSER_PN" value="634-SI8641AB-B-IS1R"/>
 <attribute name="MPN" value="SI8641AB-B-IS1R"/>
@@
 </part>
 <part name="U2" library="harp expander servo driver v1.0" deviceset="SI8641AB" device="W" package3d_urn="urn:adsk.eagle:package:16487/2" value="SI8641AB-B-IS1R">
-<attribute name="DIGIKEY_PN" value="336-5212-1-ND"/>
+<attribute name="DIGIKEY_PN" value="SI8641AB-B-IS-ND"/>
 <attribute name="MOUSER_PN" value="634-SI8641AB-B-IS1R"/>
 <attribute name="MPN" value="SI8641AB-B-IS1R"/>
@@
 <attribute name="MPN" value="IHLP2525CZER100M01"/>
 <attribute name="TYPE" value="SMD"/>
+</part>
+<part name="EXTERNAL_1" library="harp expander servo driver v1.0" deviceset="EXTERNAL" device="" value="TERMINAL BLOCK PLUG 3WAY">
+<attribute name="DIGIKEY_PN" value="732-2752-ND"/>
+<attribute name="MPN" value="691361100003"/>
+<attribute name="TYPE" value="-"/>
+</part>
+<part name="EXTERNAL_2" library="harp expander servo driver v1.0" deviceset="EXTERNAL" device="" value="TERMINAL BLOCK PLUG 3WAY">
+<attribute name="DIGIKEY_PN" value="732-2752-ND"/>
+<attribute name="MPN" value="691361100003"/>
+<attribute name="TYPE" value="-"/>
+</part>
+<part name="EXTERNAL_3" library="harp expander servo driver v1.0" deviceset="EXTERNAL" device="" value="TERMINAL BLOCK PLUG 3WAY">
+<attribute name="DIGIKEY_PN" value="732-2752-ND"/>
+<attribute name="MPN" value="691361100003"/>
+<attribute name="TYPE" value="-"/>
+</part>
+<part name="EXTERNAL_4" library="harp expander servo driver v1.0" deviceset="EXTERNAL" device="" value="CNTR PLRZD RECPT 10P">
+<attribute name="DIGIKEY_PN" value="AKC10H-ND"/>
+<attribute name="MPN" value="1658621-1"/>
+<attribute name="TYPE" value="-"/>
+</part>
+<part name="EXTERNAL_5" library="harp expander servo driver v1.0" deviceset="EXTERNAL" device="" value="CNTR PLRZD RECPT 10P">
+<attribute name="DIGIKEY_PN" value="AKC10H-ND"/>
+<attribute name="MPN" value="1658621-1"/>
+<attribute name="TYPE" value="-"/>
+</part>
+<part name="EXTERNAL_6" library="harp expander servo driver v1.0" deviceset="EXTERNAL" device="" value="10 COND. 28AWG ROUND 1PC=100FT">
+<attribute name="DIGIKEY_PN" value="3M157849-100-ND"/>
+<attribute name="MPN" value="3365/10 100"/>
+<attribute name="TYPE" value="-"/>
 </part>
 </parts>
@@
 <attribute name="TYPE" x="139.7" y="149.86" size="1.778" layer="96" rot="R90" display="off"/>
 </instance>
+<instance part="EXTERNAL_1" gate="G$1" x="160.02" y="45.72" smashed="yes">
+<attribute name="NAME" x="157.48" y="48.26" size="1.27" layer="95" font="vector" ratio="15"/>
+<attribute name="VALUE" x="157.48" y="43.18" size="1.27" layer="96" font="vector" ratio="15"/>
+<attribute name="DIGIKEY_PN" x="160.02" y="45.72" size="1.778" layer="96" display="off"/>
+</instance>
+<instance part="EXTERNAL_2" gate="G$1" x="160.02" y="38.1" smashed="yes">
+<attribute name="NAME" x="157.48" y="40.64" size="1.27" layer="95" font="vector" ratio="15"/>
+<attribute name="VALUE" x="157.48" y="35.56" size="1.27" layer="96" font="vector" ratio="15"/>
+<attribute name="DIGIKEY_PN" x="160.02" y="38.1" size="1.778" layer="96" display="off"/>
+</instance>
+<instance part="EXTERNAL_3" gate="G$1" x="160.02" y="30.48" smashed="yes">
+<attribute name="NAME" x="157.48" y="33.02" size="1.27" layer="95" font="vector" ratio="15"/>
+<attribute name="VALUE" x="157.48" y="27.94" size="1.27" layer="96" font="vector" ratio="15"/>
+<attribute name="DIGIKEY_PN" x="160.02" y="30.48" size="1.778" layer="96" display="off"/>
+</instance>
+<instance part="EXTERNAL_4" gate="G$1" x="193.04" y="45.72" smashed="yes">
+<attribute name="NAME" x="190.5" y="48.26" size="1.27" layer="95" font="vector" ratio="15"/>
+<attribute name="VALUE" x="190.5" y="43.18" size="1.27" layer="96" font="vector" ratio="15"/>
+<attribute name="DIGIKEY_PN" x="193.04" y="45.72" size="1.778" layer="96" display="off"/>
+</instance>
+<instance part="EXTERNAL_5" gate="G$1" x="193.04" y="35.56" smashed="yes">
+<attribute name="NAME" x="190.5" y="38.1" size="1.27" layer="95" font="vector" ratio="15"/>
+<attribute name="VALUE" x="190.5" y="33.02" size="1.27" layer="96" font="vector" ratio="15"/>
+<attribute name="DIGIKEY_PN" x="193.04" y="35.56" size="1.778" layer="96" display="off"/>
+</instance>
+<instance part="EXTERNAL_6" gate="G$1" x="220.98" y="45.72" smashed="yes">
+<attribute name="NAME" x="218.44" y="48.26" size="1.27" layer="95" font="vector" ratio="15"/>
+<attribute name="VALUE" x="218.44" y="43.18" size="1.27" layer="96" font="vector" ratio="15"/>
+<attribute name="DIGIKEY_PN" x="220.98" y="45.72" size="1.778" layer="96" display="off"/>
+</instance>
 </instances>
